File: KiCAD/PCB_matrix3216.kicad_sch (KiCad schematic)
At the start: 13 parts, among them IC1 NJM7805SDL1-TE1, IC2 NJM2845DL1-33-TE1, J1 Barrel_Jack_Switch, J2 Conn_02x06_Counter_Clockwise, J3 Conn_02x06_Counter_Clockwise, J4 Conn_02x02_Counter_Clockwise, J5 Conn_02x02_Counter_Clockwise, J6 Conn_01x02, U1 Matrix3216, U2 Matrix3216

Commit message: 0326
Parts:
- removed J2: Conn_02x06_Counter_Clockwise, Connector_PinHeader_2.54mm:PinHeader_2x06_P2.54mm_Horizontal, symbol Connector_Generic:Conn_02x06_Counter_Clockwise
- removed J3: Conn_02x06_Counter_Clockwise, Connector_PinSocket_2.54mm:PinSocket_2x06_P2.54mm_Horizontal, symbol Connector_Generic:Conn_02x06_Counter_Clockwise
- added C4: C, Capacitor_SMD:C_0603_1608Metric_Pad1.08x0.95mm_HandSolder, symbol Device:C
- added C5: 0.33u, Capacitor_SMD:C_0603_1608Metric_Pad1.08x0.95mm_HandSolder, symbol Device:C
- added C6: 0.1u, Capacitor_SMD:C_0603_1608Metric_Pad1.08x0.95mm_HandSolder, symbol Device:C
Connections:
- net +3.3V: now also IC2.2 (VOUT), U1.8 (IC_PWR), U2.38 (IC_PWR), C4.2, C6.1; no longer U1.18 (IC_PWR)
- net +5V: now also U1.1 (LED_PWR), U2.31 (LED_PWR); no longer U1.11 (LED_PWR)
- net GND: now also IC2.3 (GND), U1.10 (GND), U1.9 (GND), U2.39 (GND), U2.40 (GND), C4.1, C5.2, C6.2; no longer U1.19 (GND), U1.20 (GND)
- net VCC: now also IC2.1 (VIN), C5.1
- net at U2.11 (LED_PWR): no longer U1.31 (LED_PWR)
- net at U2.12 (SIN_1): no longer U1.32 (SIN_1)
- net at U2.13 (SIN_2): no longer U1.33 (SIN_2)
- net at U2.14 (SIN_3): no longer U1.34 (SIN_3)
- net at U2.15 (CLK): no longer U1.35 (CLK)
- net at U2.16 (LATCH): no longer U1.36 (LATCH)
- net at U2.17 (~{STROBE}): no longer U1.37 (~{STROBE})
- net at U2.18 (IC_PWR): no longer U1.38 (IC_PWR)
- net at U2.19 (GND): no longer U1.39 (GND)
- net at U2.20 (GND): no longer U1.40 (GND)
- net at U2.32 (SIN_1): now also U1.2 (SIN_1)
- net at U2.33 (SIN_2): now also U1.3 (SIN_2)
- net at U2.34 (SIN_3): now also U1.4 (SIN_3)
- net CLK: now reaches U2.35 (CLK)
- net CLK: now also U1.5 (CLK)
- net LATCH: now reaches U2.36 (LATCH)
- net LATCH: now also U1.6 (LATCH)
- net ~{STROBE}: now reaches U2.37 (~{STROBE})
- net ~{STROBE}: now also U1.7 (~{STROBE})
- no-connect marks 30 -> 50
Other:
- moved on the sheet: C1, C2, J5, J6, U1, U2

Commit message: schematics
Parts:
- removed C4: C, Capacitor_SMD:C_0603_1608Metric_Pad1.08x0.95mm_HandSolder, symbol Device:C
- removed J4: Conn_02x02_Counter_Clockwise, Connector_PinSocket_2.54mm:PinSocket_2x02_P2.54mm_Horizontal, symbol Connector_Generic:Conn_02x02_Counter_Clockwise
- removed J5: Conn_02x02_Counter_Clockwise, Connector_PinHeader_2.54mm:PinHeader_2x02_P2.54mm_Horizontal, symbol Connector_Generic:Conn_02x02_Counter_Clockwise
- removed J6: Conn_01x02, Connector_PinHeader_2.54mm:PinHeader_1x02_P2.54mm_Vertical, symbol Connector_Generic:Conn_01x02
- added J2: Conn_02x06_Counter_Clockwise, Connector_PinHeader_2.54mm:PinHeader_2x06_P2.54mm_Horizontal, symbol Connector_Generic:Conn_02x06_Counter_Clockwise
- added J3: Conn_02x03_Counter_Clockwise, Connector_PinHeader_2.54mm:PinHeader_2x03_P2.54mm_Horizontal, symbol Connector_Generic:Conn_02x03_Counter_Clockwise
- added J4: Conn_02x03_Counter_Clockwise, Connector_PinSocket_2.54mm:PinSocket_2x03_P2.54mm_Horizontal, symbol Connector_Generic:Conn_02x03_Counter_Clockwise
- added JP1: SolderJumper_2_Open, Jumper:SolderJumper-2_P1.3mm_Open_TrianglePad1.0x1.5mm, symbol Jumper:SolderJumper_2_Open
- C6: value 0.1u -> 2.2u
- IC2: footprint TO-252-3-L1 -> samacsys:TO-252-3-L1
- U1, U2: footprint (none) -> Library:matrix_led
Connections:
- net +3.3V: now also J2.6 (Pin_6), J2.7 (Pin_7), J4.2 (Pin_2), JP1.1 (A); no longer U2.38 (IC_PWR)
- net +5V: no longer U2.31 (LED_PWR)
- net CLK: now also J2.12 (Pin_12)
- net GND: now also J2.5 (Pin_5), J2.8 (Pin_8), J3.1 (Pin_1), J3.6 (Pin_6), J4.1 (Pin_1), J4.6 (Pin_6)
- net LATCH: now also J2.11 (Pin_11)
- net VCC: now also J3.3 (Pin_3), J3.4 (Pin_4), J4.3 (Pin_3), J4.4 (Pin_4)
- net ~{STROBE}: now also J2.10 (Pin_10)
- net SIN_1: now reaches U1.2 (SIN_1), U2.32 (SIN_1)
- net SIN_1: now also J2.1 (Pin_1)
- net SIN_2: now reaches U1.3 (SIN_2), U2.33 (SIN_2)
- net SIN_2: now also J2.2 (Pin_2)
- net SIN_3: now reaches U1.4 (SIN_3), U2.34 (SIN_3)
- net SIN_3: now also J2.3 (Pin_3)
- new net: J3.2 (Pin_2), JP1.2 (B)
- no-connect marks 50 -> 62
Other:
- moved on the sheet: C6

Commit message: Artwork
Connections:
- net CLK: now also J2.4 (Pin_4); no longer J2.12 (Pin_12)
- net SIN_2: now also J2.12 (Pin_12); no longer J2.2 (Pin_2)
- net ~{STROBE}: now also J2.2 (Pin_2); no longer J2.10 (Pin_10)
- no-connect marks 62 -> 64

Commit message: Artwork done
Connections:
- net CLK: now also J2.3 (Pin_3); no longer J2.4 (Pin_4)
- net LATCH: now also J2.2 (Pin_2); no longer J2.11 (Pin_11)
- net SIN_3: now also J2.11 (Pin_11); no longer J2.3 (Pin_3)
- net ~{STROBE}: now also J2.4 (Pin_4); no longer J2.2 (Pin_2)
Changed lines of the file:
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@@
+	(wire
+		(pts
+			(xy 78.74 175.26) (xy 84.455 175.26)
+		)
+		(stroke
+			(width 0)
+			(type default)
+		)
+	)
 	(wire
 		(pts
@@
 	(wire
 		(pts
-			(xy 78.74 175.26) (xy 84.455 175.26)
-		)
-		(stroke
-			(width 0)
-			(type default)
-		)
-	)
-	(wire
-		(pts
 			(xy 48.895 36.195) (xy 39.37 36.195)
 		)
@@
 	(wire
 		(pts
+			(xy 78.74 177.8) (xy 84.455 177.8)
+		)
+		(stroke
+			(width 0)
+			(type default)
+		)
+	)
+	(wire
+		(pts
 			(xy 102.235 93.345) (xy 107.315 93.345)
 		)
@@
 	(wire
 		(pts
+			(xy 78.74 172.72) (xy 84.455 172.72)
+		)
+		(stroke
+			(width 0)
+			(type default)
+		)
+	)
+	(wire
+		(pts
 			(xy 102.235 99.695) (xy 153.67 99.695)
 		)
@@
 	(wire
 		(pts
+			(xy 242.57 71.755) (xy 235.585 71.755)
+		)
+		(stroke
+			(width 0)
+			(type default)
+		)
+	)
+	(wire
+		(pts
+			(xy 34.925 103.505) (xy 41.275 103.505)
+		)
+		(stroke
+			(width 0)
+			(type default)
+		)
+	)
+	(wire
+		(pts
+			(xy 143.51 126.365) (xy 147.955 126.365)
+		)
+		(stroke
+			(width 0)
+			(type default)
+		)
+	)
+	(wire
+		(pts
+			(xy 127.635 36.83) (xy 127.635 37.465)
+		)
+		(stroke
+			(width 0)
+			(type default)
+		)
+	)
+	(wire
+		(pts
+			(xy 54.61 33.655) (xy 54.61 32.385)
+		)
+		(stroke
+			(width 0)
+			(type default)
+		)
+	)
+	(wire
+		(pts
+			(xy 48.895 34.29) (xy 48.895 36.195)
+		)
+		(stroke
+			(width 0)
+			(type default)
+		)
+	)
+	(wire
+		(pts
+			(xy 84.455 180.34) (xy 97.155 180.34)
+		)
+		(stroke
+			(width 0)
+			(type default)
+		)
+	)
+	(wire
+		(pts
+			(xy 84.455 180.34) (xy 68.58 180.34)
+		)
+		(stroke
+			(width 0)
+			(type default)
+		)
+	)
+	(wire
+		(pts
+			(xy 38.1 26.035) (xy 48.895 26.035)
+		)
+		(stroke
+			(width 0)
+			(type default)
+		)
+	)
+	(wire
+		(pts
+			(xy 127.635 37.465) (xy 132.08 37.465)
+		)
+		(stroke
+			(width 0)
+			(type default)
+		)
+	)
+	(wire
+		(pts
+			(xy 132.08 45.72) (xy 120.015 45.72)
+		)
+		(stroke
+			(width 0)
+			(type default)
+		)
+	)
+	(wire
+		(pts
+			(xy 87.63 26.035) (xy 87.63 29.21)
+		)
+		(stroke
+			(width 0)
+			(type default)
+		)
+	)
+	(wire
+		(pts
+			(xy 15.24 116.84) (xy 17.78 116.84)
+		)
+		(stroke
+			(width 0)
+			(type default)
+		)
+	)
+	(wire
+		(pts
+			(xy 97.155 190.5) (xy 84.455 190.5)
+		)
+		(stroke
+			(width 0)
+			(type default)
+		)
+	)
+	(wire
+		(pts
+			(xy 241.935 99.06) (xy 235.585 99.06)
+		)
+		(stroke
+			(width 0)
+			(type default)
+		)
+	)
+	(wire
+		(pts
+			(xy 39.37 31.115) (xy 34.29 31.115)
+		)
+		(stroke
+			(width 0)
+			(type default)
+		)
+	)
+	(wire
+		(pts
+			(xy 84.455 190.5) (xy 84.455 182.88)
+		)
+		(stroke
+			(width 0)
+			(type default)
+		)
+	)
+	(wire
+		(pts
+			(xy 241.935 90.17) (xy 241.935 99.06)
+		)
+		(stroke
+			(width 0)
+			(type default)
+		)
+	)
+	(wire
+		(pts
+			(xy 139.7 95.885) (xy 147.32 95.885)
+		)
+		(stroke
+			(width 0)
+			(type default)
+		)
+	)
+	(wire
+		(pts
 			(xy 97.155 172.72) (xy 101.6 172.72)
 		)
@@
 	(wire
 		(pts
-			(xy 242.57 71.755) (xy 235.585 71.755)
-		)
-		(stroke
-			(width 0)
-			(type default)
-		)
-	)
-	(wire
-		(pts
-			(xy 34.925 103.505) (xy 41.275 103.505)
-		)
-		(stroke
-			(width 0)
-			(type default)
-		)
-	)
-	(wire
-		(pts
-			(xy 143.51 126.365) (xy 147.955 126.365)
-		)
-		(stroke
-			(width 0)
-			(type default)
-		)
-	)
-	(wire
-		(pts
-			(xy 127.635 36.83) (xy 127.635 37.465)
-		)
-		(stroke
-			(width 0)
-			(type default)
-		)
-	)
-	(wire
-		(pts
-			(xy 78.74 177.8) (xy 84.455 177.8)
-		)
-		(stroke
-			(width 0)
-			(type default)
-		)
-	)
-	(wire
-		(pts
-			(xy 54.61 33.655) (xy 54.61 32.385)
-		)
-		(stroke
-			(width 0)
-			(type default)
-		)
-	)
-	(wire
-		(pts
-			(xy 48.895 34.29) (xy 48.895 36.195)
-		)
-		(stroke
-			(width 0)
-			(type default)
-		)
-	)
-	(wire
-		(pts
-			(xy 84.455 180.34) (xy 97.155 180.34)
-		)
-		(stroke
-			(width 0)
-			(type default)
-		)
-	)
-	(wire
-		(pts
-			(xy 84.455 180.34) (xy 68.58 180.34)
-		)
-		(stroke
-			(width 0)
-			(type default)
-		)
-	)
-	(wire
-		(pts
-			(xy 38.1 26.035) (xy 48.895 26.035)
-		)
-		(stroke
-			(width 0)
-			(type default)
-		)
-	)
-	(wire
-		(pts
-			(xy 78.74 172.72) (xy 84.455 172.72)
-		)
-		(stroke
-			(width 0)
-			(type default)
-		)
-	)
-	(wire
-		(pts
-			(xy 127.635 37.465) (xy 132.08 37.465)
-		)
-		(stroke
-			(width 0)
-			(type default)
-		)
-	)
-	(wire
-		(pts
-			(xy 132.08 45.72) (xy 120.015 45.72)
-		)
-		(stroke
-			(width 0)
-			(type default)
-		)
-	)
-	(wire
-		(pts
-			(xy 87.63 26.035) (xy 87.63 29.21)
-		)
-		(stroke
-			(width 0)
-			(type default)
-		)
-	)
-	(wire
-		(pts
-			(xy 15.24 116.84) (xy 17.78 116.84)
-		)
-		(stroke
-			(width 0)
-			(type default)
-		)
-	)
-	(wire
-		(pts
-			(xy 97.155 190.5) (xy 84.455 190.5)
-		)
-		(stroke
-			(width 0)
-			(type default)
-		)
-	)
-	(wire
-		(pts
-			(xy 241.935 99.06) (xy 235.585 99.06)
-		)
-		(stroke
-			(width 0)
-			(type default)
-		)
-	)
-	(wire
-		(pts
-			(xy 39.37 31.115) (xy 34.29 31.115)
-		)
-		(stroke
-			(width 0)
-			(type default)
-		)
-	)
-	(wire
-		(pts
-			(xy 84.455 190.5) (xy 84.455 182.88)
-		)
-		(stroke
-			(width 0)
-			(type default)
-		)
-	)
-	(wire
-		(pts
-			(xy 241.935 90.17) (xy 241.935 99.06)
-		)
-		(stroke
-			(width 0)
-			(type default)
-		)
-	)
-	(wire
-		(pts
-			(xy 139.7 95.885) (xy 147.32 95.885)
-		)
-		(stroke
-			(width 0)
-			(type default)
-		)
-	)
-	(wire
-		(pts
 			(xy 229.235 85.09) (xy 226.06 85.09)
 		)
@@
 	)
 	(label "CLK"
-		(at 78.74 177.8 180)
+		(at 78.74 175.26 180)
 		(effects
 			(font
@@
 	)
 	(label "~{STROBE}"
+		(at 78.74 177.8 180)
+		(effects
+			(font
+				(size 1.27 1.27)
+			)
+			(justify right bottom)
+		)
+	)
+	(label "LATCH"
 		(at 78.74 172.72 180)
 		(effects
@@
 			)
 			(justify right bottom)
-		)
-	)
-	(label "LATCH"
-		(at 101.6 172.72 0)
-		(effects
-			(font
-				(size 1.27 1.27)
-			)
-			(justify left bottom)
 		)
 	)
@@
 	)
 	(label "SIN_3"
-		(at 78.74 175.26 180)
-		(effects
-			(font
-				(size 1.27 1.27)
-			)
-			(justify right bottom)
-		)
-	)
+		(at 101.6 172.72 0)
+		(effects
+			(font
+				(size 1.27 1.27)
+			)
+			(justify left bottom)
+		)
+	)
