File: KiCAD/PCB_matrix3216.kicad_pcb (KiCad board)
At the start: 2 copper layers, 14 parts, among them IC1 NJM7805SDL1-TE1, IC2 NJM2845DL1-33-TE1, J1 Barrel_Jack_Switch, J2 Conn_02x06_Counter_Clockwise, J3 Conn_02x03_Counter_Clockwise, J4 Conn_02x03_Counter_Clockwise, U1 Matrix3216, U2 Matrix3216

Commit message: layout
Parts:
- J1: moved to B.Cu
- moved J1 52.5 mm to (188.7, 97.3), turned to 90 degrees
- moved J2 50.9 mm to (151.4, 95.1)
- moved JP1 50.7 mm to (164.5, 75.3)
- moved J4 50.7 mm to (157.4, 72.8)
- moved U2 42.7 mm to (117.3, 59.8)
- moved C2 27.6 mm to (211.4, 84.0)
- moved C6 27.6 mm to (200.5, 84.0)
- moved IC2 27.6 mm to (205.7, 91.2)
- moved C3 26.3 mm to (177.9, 84.5)
- moved C5 26.3 mm to (190.6, 84.6)
- moved IC1 26.3 mm to (184.0, 87.7)
- moved J3 13.8 mm to (216.9, 72.8)
- moved C1 0.89 mm to (188.1, 71.2)
Routing:
- net +3.3V: track 2.95 -> 6.95 mm
Other:
- board outline added: 79 x 57 mm

Commit message: update pcb layout
Parts:
- added REF**: MountingHole_3.2mm_M3, MountingHole:MountingHole_3.2mm_M3, F.Cu at (176.6, 65.4)
- added REF**: MountingHole_3.2mm_M3, MountingHole:MountingHole_3.2mm_M3, F.Cu at (168.7, 65.4)
- added REF**: MountingHole_3.2mm_M3, MountingHole:MountingHole_3.2mm_M3, F.Cu at (176.6, 113.4)
- added REF**: MountingHole_3.2mm_M3, MountingHole:MountingHole_3.2mm_M3, F.Cu at (168.7, 113.4)
- moved U2 1.00 mm to (117.2, 58.8)
- moved U1 1.00 mm to (186.7, 58.8)
Routing:
- net +3.3V: track 6.95 -> 2.95 mm
Other:
- board size 79 x 57 mm -> 79.9 x 57 mm

Commit message: Artwork
Parts:
- added REF**: PinHeader_2x06_P2.54mm_Vertical, Connector_PinHeader_2.54mm:PinHeader_2x06_P2.54mm_Vertical, F.Cu at (159.4, 102.2)
- added REF**: PinHeader_2x06_P2.54mm_Vertical, Connector_PinHeader_2.54mm:PinHeader_2x06_P2.54mm_Vertical, F.Cu at (159.4, 107.3)
- moved J3 65.7 mm to (151.4, 77.9), turned to 180 degrees
- moved J4 54.6 mm to (211.8, 77.8), turned to 180 degrees
- moved C1 1.88 mm to (187.5, 69.5)
- moved C2 0.72 mm to (210.9, 84.5)
- moved C6 0.72 mm to (200.0, 84.5)
- moved IC2 0.72 mm to (205.2, 91.7)
- turned JP1 to 180 degrees
Connections:
- J2 pad 10: /~{STROBE} -> unconnected-(J2-Pin_10-Pad10)
- J2 pad 12: /CLK -> /SIN_2
- J2 pad 2: /SIN_2 -> /~{STROBE}
- J2 pad 4: unconnected-(J2-Pin_4-Pad4) -> /CLK
Routing:
- net VCC: track 7.70 -> 153.4 mm, vias 0 -> 1
- net +3.3V: track 2.95 -> 102.9 mm, vias 0 -> 2
- net /LATCH: track 0.00 -> 90.2 mm
- net /CLK: track 0.00 -> 72.0 mm, vias 0 -> 1
- net /SIN_1: track 0.00 -> 71.8 mm
- net /SIN_2: track 0.00 -> 66.6 mm
- net /~{STROBE}: track 0.00 -> 66.5 mm, vias 0 -> 1
- net /SIN_3: track 0.00 -> 60.6 mm
- net +5V: track 3.80 -> 50.7 mm, vias 0 -> 1
- net Net-(J3-Pin_2): track 0.00 -> 11.9 mm
- net GND: vias 0 -> 23
- added copper zone on B.Cu, net GND
- added copper zone on F.Cu, net GND
Other:
- board text added: "#STROBE"
- board text added: "3V3"
- board text added: "5V"
- board text added: "8 - 30V"
- board text added: "CLK"
- board text added: "GND"
- board text added: "LATCH"
- board text added: "NJM2845DL1-33"
- board text added: "NJM7805SDL1"
- board text added: "SIN1"
- board text added: "SIN2"
- board text added: "SIN3"
- board text added: "STROBE"
- board text added: "VCC"

Commit message: artwork revise
Routing:
- net /CLK: track 72.0 -> 2.10 mm, vias 1 -> 0
- net /~{STROBE}: track 66.5 -> 5.85 mm, vias 1 -> 0
- net /LATCH: track 90.2 -> 30.8 mm
- net /SIN_3: track 60.6 -> 9.50 mm
- net /SIN_1: track 71.8 -> 25.6 mm
- net /SIN_2: track 66.6 -> 23.3 mm
- net +3.3V: track 102.9 -> 89.8 mm
Other:
- board text removed: "#STROBE"

Commit message: Artwork done
Parts:
- added REF**: TestPoint_Loop_D1.80mm_Drill1.0mm_Beaded, TestPoint:TestPoint_Loop_D1.80mm_Drill1.0mm_Beaded, F.Cu at (206.1, 79.4)
- moved C1 1.82 mm to (189.2, 69.8), turned to 90 degrees
Connections:
- J2 pad 11: /LATCH -> /SIN_3
- J2 pad 2: /~{STROBE} -> /LATCH
- J2 pad 3: /SIN_3 -> /CLK
- J2 pad 4: /CLK -> /~{STROBE}
- REF** pad 2: (no net) -> +3.3V
- REF** pad 4: (no net) -> GND
Routing:
- net /~{STROBE}: track 5.85 -> 82.7 mm, vias 0 -> 1
- net /CLK: track 2.10 -> 60.4 mm
- net /SIN_3: track 9.50 -> 54.4 mm, vias 0 -> 1
- net /SIN_2: track 23.3 -> 63.7 mm
- net /LATCH: track 30.8 -> 66.0 mm, vias 0 -> 1
- net /SIN_1: track 25.6 -> 58.7 mm
- net +3.3V: track 89.8 -> 113.3 mm
- net +5V: track 50.7 -> 67.7 mm
- net GND: track 0.00 -> 2.29 mm, vias 23 -> 26
Other:
- board text added: "秋月ドット抜けマトリクス"

Commit message: pcb done
Other:
- board text added: "秋月ドット抜けマトリクスLED"
- board text removed: "秋月ドット抜けマトリクス"
Changed lines of the file:
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@@
 			(outputformat 1)
 			(mirror no)
-			(drillshape 1)
+			(drillshape 0)
 			(scaleselection 1)
-			(outputdirectory "")
+			(outputdirectory "output/")
 		)
 	)
@@
 		)
 	)
-	(gr_text "秋月ドット抜けマトリクス"
-		(at 208.407 115.697 0)
+	(gr_text "秋月ドット抜けマトリクスLED"
+		(at 206.3242 115.8494 0)
 		(layer "F.SilkS")
 		(effects
